Commit message: Fix hardware error

File: description/ros2_control.xacro (robot description, xacro)
@@ -18,6 +18,6 @@
                     <param name="max">10</param>
                 </command_interface>
+                <state_interface name="position"/>
                 <state_interface name="velocity"/>
-                <state_interface name="position"/>
             </joint>
             <joint name="right_wheel_joint">
@@ -26,6 +26,6 @@
                     <param name="max">10</param>
                 </command_interface>
+                <state_interface name="position"/>
                 <state_interface name="velocity"/>
-                <state_interface name="position"/>
             </joint>
         </ros2_control>
@@ -36,21 +36,21 @@
                 <plugin>gazebo_ros2_control/GazeboSystem</plugin>
             </hardware>
-            <joint name="left_wheel_joint">
-                <command_interface name="velocity">
-                    <param name="min">-10</param>
-                    <param name="max">10</param>
-                </command_interface>
-                <state_interface name="velocity"/>
-                <state_interface name="position"/>
-            </joint>
-            <joint name="right_wheel_joint">
-                <command_interface name="velocity">
-                    <param name="min">-10</param>
-                    <param name="max">10</param>
-                </command_interface>
-                <state_interface name="velocity"/>
-                <state_interface name="position"/>
-            </joint>
-        </ros2_control>
+        <joint name="left_wheel_joint">
+            <command_interface name="velocity">
+                <param name="min">-10</param>
+                <param name="max">10</param>
+            </command_interface>
+            <state_interface name="position"/>
+            <state_interface name="velocity"/>
+        </joint>
+        <joint name="right_wheel_joint">
+            <command_interface name="velocity">
+                <param name="min">-10</param>
+                <param name="max">10</param>
+            </command_interface>
+            <state_interface name="position"/>
+            <state_interface name="velocity"/>
+        </joint>
+    </ros2_control>
     </xacro:if>
      <gazebo>
